Commit message: 1

File: urdf/robot_core.xacro (robot description, xacro)
@@ -28,5 +28,5 @@
             <origin xyz="0 0 0" rpy="0 0 0"/>
             <geometry>
-                <mesh   filename="package://AMR-Sweeper_description/meshes/Chassis/Chassis.stl" />
+                <mesh   filename="package://amr-sweeper_description/meshes/Chassis/Chassis.stl" />
             </geometry>
         </collision>
@@ -48,5 +48,5 @@
             <origin xyz="0 0 0" rpy="${pi/2} 0 0"/>
             <geometry>
-                <mesh   filename="package://AMR-Sweeper_description/meshes/WheelAssembly/WheelAssembly.stl" />
+                <mesh   filename="package://amr-sweeper_description/meshes/WheelAssembly/WheelAssembly.stl" />
             </geometry>
             <material name="yellow"/>
@@ -55,5 +55,5 @@
             <origin xyz="0 0 0" rpy="${pi/2} 0 0"/>
             <geometry>
-                <mesh   filename="package://AMR-Sweeper_description/meshes/WheelAssembly/WheelAssembly.stl" />
+                <mesh   filename="package://amr-sweeper_description/meshes/WheelAssembly/WheelAssembly.stl" />
             </geometry>
         </collision>
@@ -74,5 +74,5 @@
             <origin xyz="0 0 0" rpy="${pi/2} 0 0"/>
             <geometry>
-                <mesh   filename="package://AMR-Sweeper_description/meshes/WheelAssembly/WheelAssembly.stl" />
+                <mesh   filename="package://amr-sweeper_description/meshes/WheelAssembly/WheelAssembly.stl" />
             </geometry>
             <material name="yellow"/>
@@ -81,5 +81,5 @@
             <origin xyz="0 0 0" rpy="${pi/2} 0 0"/>
             <geometry>
-                <mesh   filename="package://AMR-Sweeper_description/meshes/WheelAssembly/WheelAssembly.stl" />
+                <mesh   filename="package://amr-sweeper_description/meshes/WheelAssembly/WheelAssembly.stl" />
             </geometry>
         </collision>
@@ -101,5 +101,5 @@
             <origin xyz="0 0 0" rpy="0 0 0"/>
             <geometry>
-                <mesh   filename="package://AMR-Sweeper_description/meshes/Tool/Tool.stl" />
+                <mesh   filename="package://amr-sweeper_description/meshes/Tool/Tool.stl" />
             </geometry>
             <material name="black"/>
@@ -120,5 +120,5 @@
             <origin xyz="0 0 0" rpy="0 0 0"/>
             <geometry>
-                <mesh   filename="package://AMR-Sweeper_description/meshes/Tool/Brush.stl" />
+                <mesh   filename="package://amr-sweeper_description/meshes/Tool/Brush.stl" />
             </geometry>
             <material name="red"/>
@@ -127,5 +127,5 @@
             <origin xyz="0 0 0" rpy="0 0 0"/>
             <geometry>
-                <mesh   filename="package://AMR-Sweeper_description/meshes/Tool/Brush.stl" />
+                <mesh   filename="package://amr-sweeper_description/meshes/Tool/Brush.stl" />
             </geometry>
         </collision>
@@ -145,5 +145,5 @@
             <origin xyz="0 0 0" rpy="0 0 0"/>
             <geometry>
-                <mesh   filename="package://AMR-Sweeper_description/meshes/Tool/Brush.stl" />
+                <mesh   filename="package://amr-sweeper_description/meshes/Tool/Brush.stl" />
             </geometry>
             <material name="red"/>
@@ -152,5 +152,5 @@
             <origin xyz="0 0 0" rpy="0 0 0"/>
             <geometry>
-                <mesh   filename="package://AMR-Sweeper_description/meshes/Tool/Brush.stl" />
+                <mesh   filename="package://amr-sweeper_description/meshes/Tool/Brush.stl" />
             </geometry>
         </collision>

Commit message: 2

File: urdf/robot_core.xacro (robot description, xacro)
@@ -19,5 +19,5 @@
             <origin xyz="0 0 0" rpy="0 0 0"/>
             <geometry>
-                <mesh   filename="package://amr-sweeper_description/meshes/chassis/chassis.stl"
+                <mesh   filename="package://amr-sweeper_description/meshes/chassis/chassis.dae"
                         scale="0.001 0.001 0.001" />
             </geometry>

Commit message: 3

File: urdf/robot_core.xacro (robot description, xacro)
@@ -10,10 +10,10 @@
     <link name="base_footprint">
     </link>
-    <joint name="Chassis_joint" type="fixed">
+    <joint name="chassis_joint" type="fixed">
         <parent link="base_link" />
-        <child  link="Chassis_link" />
+        <child  link="chassis_link" />
         <origin xyz="0 0 0" rpy="0 0 0"/>
     </joint>
-    <link name="Chassis_link">
+    <link name="chassis_link">
         <visual>
             <origin xyz="0 0 0" rpy="0 0 0"/>

Commit message: 4

File: urdf/robot_core.xacro (robot description, xacro)
@@ -19,5 +19,5 @@
             <origin xyz="0 0 0" rpy="0 0 0"/>
             <geometry>
-                <mesh   filename="package://amr-sweeper_description/meshes/chassis/chassis.dae"
+                <mesh   filename="package://amrsweeper_description/meshes/chassis/chassis.dae"
                         scale="0.001 0.001 0.001" />
             </geometry>
@@ -28,5 +28,5 @@
             <origin xyz="0 0 0" rpy="0 0 0"/>
             <geometry>
-                <mesh   filename="package://amr-sweeper_description/meshes/Chassis/Chassis.stl" />
+                <mesh   filename="package://amrsweeper_description/meshes/Chassis/Chassis.stl" />
             </geometry>
         </collision>
@@ -48,5 +48,5 @@
             <origin xyz="0 0 0" rpy="${pi/2} 0 0"/>
             <geometry>
-                <mesh   filename="package://amr-sweeper_description/meshes/WheelAssembly/WheelAssembly.stl" />
+                <mesh   filename="package://amrsweeper_description/meshes/WheelAssembly/WheelAssembly.stl" />
             </geometry>
             <material name="yellow"/>
@@ -55,5 +55,5 @@
             <origin xyz="0 0 0" rpy="${pi/2} 0 0"/>
             <geometry>
-                <mesh   filename="package://amr-sweeper_description/meshes/WheelAssembly/WheelAssembly.stl" />
+                <mesh   filename="package://amrsweeper_description/meshes/WheelAssembly/WheelAssembly.stl" />
             </geometry>
         </collision>
@@ -74,5 +74,5 @@
             <origin xyz="0 0 0" rpy="${pi/2} 0 0"/>
             <geometry>
-                <mesh   filename="package://amr-sweeper_description/meshes/WheelAssembly/WheelAssembly.stl" />
+                <mesh   filename="package://amrsweeper_description/meshes/WheelAssembly/WheelAssembly.stl" />
             </geometry>
             <material name="yellow"/>
@@ -81,5 +81,5 @@
             <origin xyz="0 0 0" rpy="${pi/2} 0 0"/>
             <geometry>
-                <mesh   filename="package://amr-sweeper_description/meshes/WheelAssembly/WheelAssembly.stl" />
+                <mesh   filename="package://amrsweeper_description/meshes/WheelAssembly/WheelAssembly.stl" />
             </geometry>
         </collision>
@@ -101,5 +101,5 @@
             <origin xyz="0 0 0" rpy="0 0 0"/>
             <geometry>
-                <mesh   filename="package://amr-sweeper_description/meshes/Tool/Tool.stl" />
+                <mesh   filename="package://amrsweeper_description/meshes/Tool/Tool.stl" />
             </geometry>
             <material name="black"/>
@@ -120,5 +120,5 @@
             <origin xyz="0 0 0" rpy="0 0 0"/>
             <geometry>
-                <mesh   filename="package://amr-sweeper_description/meshes/Tool/Brush.stl" />
+                <mesh   filename="package://amrsweeper_description/meshes/Tool/Brush.stl" />
             </geometry>
             <material name="red"/>
@@ -127,5 +127,5 @@
             <origin xyz="0 0 0" rpy="0 0 0"/>
             <geometry>
-                <mesh   filename="package://amr-sweeper_description/meshes/Tool/Brush.stl" />
+                <mesh   filename="package://amrsweeper_description/meshes/Tool/Brush.stl" />
             </geometry>
         </collision>
@@ -145,5 +145,5 @@
             <origin xyz="0 0 0" rpy="0 0 0"/>
             <geometry>
-                <mesh   filename="package://amr-sweeper_description/meshes/Tool/Brush.stl" />
+                <mesh   filename="package://amrsweeper_description/meshes/Tool/Brush.stl" />
             </geometry>
             <material name="red"/>
@@ -152,5 +152,5 @@
             <origin xyz="0 0 0" rpy="0 0 0"/>
             <geometry>
-                <mesh   filename="package://amr-sweeper_description/meshes/Tool/Brush.stl" />
+                <mesh   filename="package://amrsweeper_description/meshes/Tool/Brush.stl" />
             </geometry>
         </collision>

Commit message: 5

File: urdf/robot_core.xacro (robot description, xacro)
@@ -19,5 +19,5 @@
             <origin xyz="0 0 0" rpy="0 0 0"/>
             <geometry>
-                <mesh   filename="package://amrsweeper_description/meshes/chassis/chassis.dae"
+                <mesh   filename="package://amrsweeper_description/meshes/chassis/chassis.stl"
                         scale="0.001 0.001 0.001" />
             </geometry>
